Commit message: Created gripper_communication package, added new bringup and ros control launch files, made small changes to description files.

File: ur5_gripper/description/urdf/ur5_gripper_robot.urdf.xacro (robot description, xacro)
@@ -12,6 +12,4 @@
   <!-- robotiq_ft300-->
   <xacro:include filename="$(find robotiq_ft_sensor)/urdf/robotiq_ft300.urdf.xacro" />
-  <!-- kinect with plugin-->
-  <xacro:include filename="$(find common_sensors)/urdf/sensors/kinect2.urdf.xacro" />
   <xacro:include filename="$(find robotiq_2f_140_gripper_visualization)/urdf/robotiq140_plugin.xacro" />
   <!-- arm -->
@@ -28,13 +26,4 @@
   <xacro:robotiq_arg2f_140 prefix=""/>
   <link name="world" />
-  <xacro:kinect2  parent="world" name="kinectv2_1" >
-    <origin xyz="1.5 0.6 1.0" rpy="0.0 0.30 3.0" />
-  </xacro:kinect2>
-  <xacro:kinect2  parent="world" name="kinectv2_2" >
-    <origin xyz="-0.7 0 1.0" rpy="0 0.15 1.5" />
-  </xacro:kinect2>
-  <xacro:kinect2  parent="world" name="kinectv2_3" >
-    <origin xyz="1.4 0.0 1.6" rpy="0.0 0.8 2.70" />
-  </xacro:kinect2>
   <joint name="world_joint" type="fixed">
     <parent link="world" />

Commit message: Added gripper communication.

File: ur5_gripper/description/urdf/ur5_gripper_robot.urdf.xacro (robot description, xacro)
@@ -30,4 +30,5 @@
     <child link = "base_link" />
     <origin xyz="0.0 0.0 1.1" rpy="0.0 0.0 0.0" />
+    <!-- <origin xyz="0.0 0.0 0.0" rpy="0.0 0.0 0.0" /> -->
   </joint>
   <!-- sensor -->
